Commit message: changed endeffector joint to prismatic joint with no range -> end_effector can now be found in the gazebo Poses topic -> really dirty, but works for now

File: open_manipulator_x_description/urdf/open_manipulator_x.transmission.xacro (robot description, xacro)
@@ -38,4 +38,19 @@
     </ros2_control>
   </xacro:macro>
+  <!-- <xacro:macro name="Ros2ControlFixedJoint" params="joint n">
+    <ros2_control name="control${n}" type="system">
+      <hardware>
+        <plugin>ign_ros2_control/IgnitionSystem</plugin>
+      </hardware>
+      <joint name="${joint}">
+        <state_interface name="position">
+          <param name="initial_value">0.0</param>
+        </state_interface>
+        <state_interface name="velocity">
+          <param name="initial_value">0.0</param>
+        </state_interface>
+      </joint>
+    </ros2_control>
+  </xacro:macro> -->
   <!-- ros2_control for joint1 -->
   <xacro:Ros2ControlPositionJoint n="1" joint="joint1" />
@@ -50,4 +65,6 @@
   <!-- ros2_control for gripper_sub -->
   <xacro:Ros2ControlEffortJoint n="6" joint="gripper_sub" />
+    <!-- ros2_control for end_effector_joint -->
+  <xacro:Ros2ControlPositionJoint n="7" joint="end_effector_joint"/>
 </robot>
 <!-- <?xml version="1.0"?>

File: open_manipulator_x_description/urdf/open_manipulator_x.urdf.xacro (robot description, xacro)
@@ -219,8 +219,10 @@
   </link>
   <!-- end effector joint -->
-  <joint name="end_effector_joint" type="fixed">
+  <joint name="end_effector_joint" type="prismatic">
     <origin xyz="0.126 0.0 0.0" rpy="0 0 0"/>
     <parent link="link5"/>
     <child link="end_effector_link"/>
+    <axis xyz="0 1 0"/>
+    <limit velocity="0.0" effort="1" lower="0.0" upper="0.0" />
   </joint>
   <!-- end effector link -->
