Commit message: changed friction values of gripper links -> cube graspable

File: open_manipulator_x_description/urdf/open_manipulator_x.urdf.xacro (robot description, xacro)
@@ -161,5 +161,5 @@
     <origin xyz="0.0817 0.021 0.0" rpy="0 0 0"/>
     <axis xyz="0 1 0"/>
-    <limit velocity="4.8" effort="1" lower="-0.010" upper="0.019" />
+    <limit velocity="4.8" effort="100" lower="-0.010" upper="0.019" />
   </joint>
   <!--  Gripper link -->
@@ -177,4 +177,12 @@
         <mesh filename="package://chain_link_grip_l.stl" scale="0.001 0.001 0.001"/>
       </geometry>
+      <surface>
+        <friction>
+          <ode>
+            <mu>100000.0</mu>
+            <mu2>100000.0</mu2>
+          </ode>
+        </friction>
+      </surface>
     </collision>
     <inertial>
@@ -192,5 +200,5 @@
     <origin xyz="0.0817 -0.021 0.0" rpy="0 0 0"/>
     <axis xyz="0 -1 0"/>
-    <limit velocity="4.8" effort="1" lower="-0.010" upper="0.019" />
+    <limit velocity="4.8" effort="100" lower="-0.010" upper="0.019" />
     <mimic joint="gripper" multiplier="1"/>
   </joint>
@@ -209,4 +217,12 @@
         <mesh filename="package://chain_link_grip_r.stl" scale="0.001 0.001 0.001"/>
       </geometry>
+      <surface>
+        <friction>
+          <ode>
+            <mu>100000.0</mu>
+            <mu2>100000.0</mu2>
+          </ode>
+        </friction>
+      </surface>
     </collision>
     <inertial>
@@ -224,5 +240,5 @@
     <child link="end_effector_link"/>
     <axis xyz="0 1 0"/>
-    <limit velocity="0.0" effort="1" lower="0.0" upper="0.0" />
+    <limit velocity="4.8" effort="1" lower="0.0" upper="0.01" />
   </joint>
   <!-- end effector link -->
